File: LoRaWAN-HelloWorld-radiolib/KiCAD/ESP32-LoRa-SX1262/ESP32-LoRa-SX1262.kicad_sch (KiCad schematic)
At the start: 6 parts, among them U1 Gravity TDS Meter, U2 SX1262IMLTRT, U3 LEA-M8T, U4 PH Module Logo-Rnaenaor V2.0, U5 ESP32-DEVKITC-32UE, U6 LGZD Sensor v1.1

Commit message: Modernize
Connections:
- net at U6. (4): now also U5.8 (33)
Other:
- title: ESP32-WROOM-32 | SX1262 -> ESP32 NodeMCU | SX1262 + Sensors
